Commit message: Add collisions

File: urdf/cassie_v4.urdf (robot description, URDF)
Before this commit: robot cassie_v4, 17 links, 16 joints
Links:
- link leftfoot: geometry collision mesh filename=package://cassie_description/meshes/left-foot.stl scale=1 1 1; visual mesh filename=package://cassie_description/meshes/left-foot.stl scale=1 1 1
- link leftheelspring: geometry collision mesh filename=package://cassie_description/meshes/left-heel-spring.stl scale=1 1 1; visual mesh filename=package://cassie_description/meshes/left-heel-spring.stl scale=1 1 1
- link lefthippitch: geometry collision mesh filename=package://cassie_description/meshes/LeftHipPitch.stl scale=1 1 1; visual mesh filename=package://cassie_description/meshes/LeftHipPitch.stl scale=1 1 1
- link lefthiproll: geometry collision mesh filename=package://cassie_description/meshes/LeftHipRoll.stl scale=1 1 1; visual mesh filename=package://cassie_description/meshes/LeftHipRoll.stl scale=1 1 1
- link lefthipyaw: geometry collision mesh filename=package://cassie_description/meshes/LeftHipYaw.stl scale=1 1 1; visual mesh filename=package://cassie_description/meshes/LeftHipYaw.stl scale=1 1 1
- link leftknee: geometry collision mesh filename=package://cassie_description/meshes/left-knee.stl scale=1 1 1; visual mesh filename=package://cassie_description/meshes/left-knee.stl scale=1 1 1
- link leftshin: geometry collision mesh filename=package://cassie_description/meshes/left-shin.stl scale=1 1 1; visual mesh filename=package://cassie_description/meshes/left-shin.stl scale=1 1 1
- link lefttarsus: geometry collision mesh filename=package://cassie_description/meshes/left-tarsus.stl scale=1 1 1; visual mesh filename=package://cassie_description/meshes/left-tarsus.stl scale=1 1 1
- link pelvis: geometry collision mesh filename=package://cassie_description/meshes/cassie-pelvis.stl scale=1 1 1; visual mesh filename=package://cassie_description/meshes/cassie-pelvis.stl scale=1 1 1
- link rightfoot: geometry collision mesh filename=package://cassie_description/meshes/right-foot.stl scale=1 1 1; visual mesh filename=package://cassie_description/meshes/right-foot.stl scale=1 1 1
- link rightheelspring: geometry collision mesh filename=package://cassie_description/meshes/left-heel-spring.stl scale=1 1 1; visual mesh filename=package://cassie_description/meshes/left-heel-spring.stl scale=1 1 1
- link righthippitch: geometry collision mesh filename=package://cassie_description/meshes/RightHipPitch.stl scale=1 1 1; visual mesh filename=package://cassie_description/meshes/RightHipPitch.stl scale=1 1 1
- link righthiproll: geometry collision mesh filename=package://cassie_description/meshes/RightHipRoll.stl scale=1 1 1; visual mesh filename=package://cassie_description/meshes/RightHipRoll.stl scale=1 1 1
- link righthipyaw: geometry collision mesh filename=package://cassie_description/meshes/RightHipYaw.stl scale=1 1 1; visual mesh filename=package://cassie_description/meshes/RightHipYaw.stl scale=1 1 1
- link rightknee: geometry collision mesh filename=package://cassie_description/meshes/right-knee.stl scale=1 1 1; visual mesh filename=package://cassie_description/meshes/right-knee.stl scale=1 1 1
- link rightshin: geometry collision mesh filename=package://cassie_description/meshes/right-shin.stl scale=1 1 1; visual mesh filename=package://cassie_description/meshes/right-shin.stl scale=1 1 1
- link righttarsus: geometry collision mesh filename=package://cassie_description/meshes/right-tarsus.stl scale=1 1 1; visual mesh filename=package://cassie_description/meshes/right-tarsus.stl scale=1 1 1
